Commit message: navigation stack

File: diy_robot/src/jst_laser/urdf/robot1_base_04.xacro (robot description, xacro)
@@ -192,5 +192,5 @@
       <origin xyz="0 0 0" rpy="0 0 0"/>
       <geometry>
-        <mesh filename="hokuyo.dae"/>
+        <mesh filename="package://jst_laser/meshes/hokuyo.dae"/>
       </geometry>
     </visual>
